Commit message: KIRO snake urdf added and gazebo ready!

File: src/snake_description/urdf/quadnake_ver_leg.urdf (robot description, URDF)
Before this commit: robot quadnake_ver_leg, 9 links, 8 joints
Links:
- removed link Link0
- removed link base_footprint
- added link base_link, mass 0.52162; collision mesh filename=package://snake_description/meshes/quadnake/base_link.STL; visual mesh filename=package://snake_description/meshes/quadnake/base_link.STL
- link Link1: geometry collision mesh filename=package://snake_description/meshes/quadnake/Link1.STL; visual mesh filename=package://snake_description/meshes/quadnake/Link1.STL
- link Link2: geometry collision mesh filename=package://snake_description/meshes/quadnake/Link2.STL; visual mesh filename=package://snake_description/meshes/quadnake/Link2.STL
- link Link3: geometry collision mesh filename=package://snake_description/meshes/quadnake/Link3.STL; visual mesh filename=package://snake_description/meshes/quadnake/Link3.STL
- link Link4: geometry collision mesh filename=package://snake_description/meshes/quadnake/Link4.STL; visual mesh filename=package://snake_description/meshes/quadnake/Link4.STL
- link Link5: geometry collision mesh filename=package://snake_description/meshes/quadnake/Link5.STL; visual mesh filename=package://snake_description/meshes/quadnake/Link5.STL
- link Link6: geometry collision mesh filename=package://snake_description/meshes/quadnake/Link6.STL; visual mesh filename=package://snake_description/meshes/quadnake/Link6.STL
- link Link7: geometry collision mesh filename=package://snake_description/meshes/quadnake/Link7.STL; visual mesh filename=package://snake_description/meshes/quadnake/Link7.STL
Joints:
- removed joint base_link_joint
- joint Joint1: parent Link0 -> base_link
